Commit message: Replaced bus_loki.urdf with Rohan's version.

File: urdf/bus_loki.urdf (robot description, URDF)
Before this commit: robot test_robot, 4 links, 3 joints
Links:
- removed link link1
- removed link link2
- removed link link3
- removed link link4
- added link base_link
- added link sonar_0
- added link sonar_1
- added link sonar_10
- added link sonar_11
- added link sonar_12
- added link sonar_13
- added link sonar_14
- added link sonar_15
- added link sonar_2
- added link sonar_3
- added link sonar_4
- added link sonar_5
- added link sonar_6
- added link sonar_7
- added link sonar_8
- added link sonar_9
Joints:
- removed joint joint1
- removed joint joint2
- removed joint joint3
- added joint base_sonar_0: type fixed, parent base_link, child sonar_0, origin xyz=0.088 0 0 rpy=0 0 0
- added joint base_sonar_1: type fixed, parent base_link, child sonar_1, origin xyz=0.0838134 0.0210476 0 rpy=0 0 0.39
- added joint base_sonar_10: type fixed, parent base_link, child sonar_10, origin xyz=-0.155890873 -0.038890873 0 rpy=0 0 -2.35619449
- added joint base_sonar_11: type fixed, parent base_link, child sonar_11, origin xyz=-0.138047589 -0.050813374 0 rpy=0 0 -1.96349541
- added joint base_sonar_12: type fixed, parent base_link, child sonar_12, origin xyz=-0.117 -0.055 0 rpy=0 0 -1.57
- added joint base_sonar_13: type fixed, parent base_link, child sonar_13, origin xyz=0.0540476 -0.0508134 0 rpy=0 0 -1.17
- added joint base_sonar_14: type fixed, parent base_link, child sonar_14, origin xyz=0.0718909 -0.0388909 0 rpy=0 0 -0.79
- added joint base_sonar_15: type fixed, parent base_link, child sonar_15, origin xyz=0.0838134 -0.0210476 0 rpy=0 0 -0.39
- added joint base_sonar_2: type fixed, parent base_link, child sonar_2, origin xyz=0.0718909 0.0388909 0 rpy=0 0 0.79
- added joint base_sonar_3: type fixed, parent base_link, child sonar_3, origin xyz=0.0540476 0.0508134 0 rpy=0 0 1.17
- added joint base_sonar_4: type fixed, parent base_link, child sonar_4, origin xyz=-0.117 0.055 0 rpy=0 0 1.57
- added joint base_sonar_5: type fixed, parent base_link, child sonar_5, origin xyz=-0.138047589 0.050813374 0 rpy=0 0 1.96349541
- added joint base_sonar_6: type fixed, parent base_link, child sonar_6, origin xyz=-0.155890873 0.038890873 0 rpy=0 0 2.35619449
- added joint base_sonar_7: type fixed, parent base_link, child sonar_7, origin xyz=-0.167813374 0.021047589 0 rpy=0 0 2.74889357
- added joint base_sonar_8: type fixed, parent base_link, child sonar_8, origin xyz=-0.172 0 0 rpy=0 0 3.14159265
- added joint base_sonar_9: type fixed, parent base_link, child sonar_9, origin xyz=-0.167813374 -0.021047589 0 rpy=0 0 -2.74889357

Commit message: Updated the use consistent numbers for the sonars.  They should match the my_arduino_params.yaml.loki file.

File: urdf/bus_loki.urdf (robot description, URDF)
Before this commit: robot loki, 17 links, 16 joints
Links:
- removed link sonar_0
- added link sonar_16
Joints:
- removed joint base_sonar_0
- added joint base_sonar_16: type fixed, parent base_link, child sonar_16, origin xyz=0.0838134 -0.0210476 0 rpy=0 0 -0.39
- joint base_sonar_1: origin xyz=0.0838134 0.0210476 0 rpy=0 0 0.39 -> xyz=0.088 0 0 rpy=0 0 0
- joint base_sonar_10: origin xyz=-0.155890873 -0.038890873 0 rpy=0 0 -2.35619449 -> xyz=-0.167813374 -0.021047589 0 rpy=0 0 -2.74889357
- joint base_sonar_11: origin xyz=-0.138047589 -0.050813374 0 rpy=0 0 -1.96349541 -> xyz=-0.155890873 -0.038890873 0 rpy=0 0 -2.35619449
- joint base_sonar_12: origin xyz=-0.117 -0.055 0 rpy=0 0 -1.57 -> xyz=-0.138047589 -0.050813374 0 rpy=0 0 -1.96349541
- joint base_sonar_13: child sonar_13 -> sonar_12; origin xyz=0.0540476 -0.0508134 0 rpy=0 0 -1.17 -> xyz=-0.117 -0.055 0 rpy=0 0 -1.57
- joint base_sonar_14: origin xyz=0.0718909 -0.0388909 0 rpy=0 0 -0.79 -> xyz=0.0540476 -0.0508134 0 rpy=0 0 -1.17
- joint base_sonar_15: origin xyz=0.0838134 -0.0210476 0 rpy=0 0 -0.39 -> xyz=0.0718909 -0.0388909 0 rpy=0 0 -0.79
- joint base_sonar_2: origin xyz=0.0718909 0.0388909 0 rpy=0 0 0.79 -> xyz=0.0838134 0.0210476 0 rpy=0 0 0.39
- joint base_sonar_3: origin xyz=0.0540476 0.0508134 0 rpy=0 0 1.17 -> xyz=0.0718909 0.0388909 0 rpy=0 0 0.79
- joint base_sonar_4: origin xyz=-0.117 0.055 0 rpy=0 0 1.57 -> xyz=0.0540476 0.0508134 0 rpy=0 0 1.17
- joint base_sonar_5: origin xyz=-0.138047589 0.050813374 0 rpy=0 0 1.96349541 -> xyz=-0.117 0.055 0 rpy=0 0 1.57
- joint base_sonar_6: origin xyz=-0.155890873 0.038890873 0 rpy=0 0 2.35619449 -> xyz=-0.138047589 0.050813374 0 rpy=0 0 1.96349541
- joint base_sonar_7: origin xyz=-0.167813374 0.021047589 0 rpy=0 0 2.74889357 -> xyz=-0.155890873 0.038890873 0 rpy=0 0 2.35619449
- joint base_sonar_8: origin xyz=-0.172 0 0 rpy=0 0 3.14159265 -> xyz=-0.167813374 0.021047589 0 rpy=0 0 2.74889357
- joint base_sonar_9: origin xyz=-0.167813374 -0.021047589 0 rpy=0 0 -2.74889357 -> xyz=-0.172 0 0 rpy=0 0 3.14159265

Commit message: Fixed bug in URDF file.

File: urdf/bus_loki.urdf (robot description, URDF)
Before this commit: robot loki, 17 links, 16 joints
Joints:
- joint base_sonar_13: child sonar_12 -> sonar_13
